File: V2 SMD/Hardware/Water Tank Sensor V2.kicad_pcb (KiCad board)
At the start: 2 copper layers, 24 parts, among them J1 Valve Terminal, J2 Temp Sensor, J3 Water Level Sensor, J4 12v in, Q1 AO3400A, U1 ESP32-WROOM-32D, U2 AMS1117-3.3

Commit message: Added schematic image
Parts:
- removed C1: 1uF, Capacitor_SMD:C_0805_2012Metric
- removed C2, C4: 10uF, Capacitor_SMD:C_0805_2012Metric
- removed C3: 0.1uF, Capacitor_SMD:C_0805_2012Metric
- removed C5, C6, C7: 22uF, Capacitor_SMD:C_0805_2012Metric
- removed D1: 1N4148W, Diode_SMD:D_SOD-123
- removed D2: Red LED, LED_SMD:LED_0805_2012Metric
- removed J1: Valve Terminal, TerminalBlock_Phoenix:TerminalBlock_Phoenix_MKDS-1,5-3_1x03_P5.00mm_Horizontal
- removed J2: Temp Sensor, Connector_JST:JST_XH_B3B-XH-A_1x03_P2.50mm_Vertical
- removed J3: Water Level Sensor, Connector_JST:JST_XH_B2B-XH-A_1x02_P2.50mm_Vertical
- removed J4: 12v in, TerminalBlock_Phoenix:TerminalBlock_Phoenix_MKDS-1,5-2_1x02_P5.00mm_Horizontal
- removed PS1: K7805-500R3, SamacSys_Parts:K7805500R3
- removed Q1: AO3400A, Package_TO_SOT_SMD:SOT-23
- removed R1, R3: 470, Resistor_SMD:R_0805_2012Metric
- removed R2: 47k, Resistor_SMD:R_0805_2012Metric
- removed R4: 4.7k, Resistor_SMD:R_0805_2012Metric
- removed R5: 10k, Resistor_SMD:R_0805_2012Metric
- removed R6: 2k, Resistor_SMD:R_0805_2012Metric
- removed Relay1: Relay, Relay_THT:Relay_SPDT_SANYOU_SRD_Series_Form_C
- removed U1: ESP32-WROOM-32D, RF_Module:ESP32-WROOM-32
- removed U2: AMS1117-3.3, Package_TO_SOT_SMD:SOT-223-3_TabPin2
Routing:
- net VDD33: track 25.0 -> 0.00 mm
- net Temp: track 11.8 -> 0.00 mm, vias 2 -> 0
- net ADC1: track 2.58 -> 0.00 mm

Commit message: Added completed PCB layout for V2SMD with images
Parts:
- added C1: 10uF, Capacitor_SMD:C_0805_2012Metric, F.Cu at (112.0, 103.5)
- added C2: 22uF, Capacitor_SMD:C_0805_2012Metric, F.Cu at (92.9, 103.5)
- added C3: 22uF, Capacitor_SMD:C_0805_2012Metric, F.Cu at (90.4, 103.5)
- added C4: 22uF, Capacitor_SMD:C_0805_2012Metric, F.Cu at (87.9, 103.5)
- added C5: 1uF, Capacitor_SMD:C_0805_2012Metric, F.Cu at (88.0, 85.3)
- added C6: 10uF, Capacitor_SMD:C_0805_2012Metric, F.Cu at (90.8, 60.5)
- added C7: 0.1uF, Capacitor_SMD:C_0805_2012Metric, F.Cu at (92.9, 60.5)
- added D1: SS14, SamacSys_Parts:DIOM5126X250N, F.Cu at (83.4, 87.8)
- added D2: SS14, SamacSys_Parts:DIOM5126X250N, F.Cu at (112.0, 98.5)
- added D3: Red LED, LED_SMD:LED_0805_2012Metric, F.Cu at (88.9, 90.7)
- added D4: 1N4148W, Diode_SMD:D_SOD-123, F.Cu at (93.4, 90.0)
- added D5: Red LED, LED_SMD:LED_0805_2012Metric, F.Cu at (92.4, 112.0)
- added G***: LOGO, logos:smartrv, F.Cu at (88.2, 67.0)
- added G***: LOGO, logos:qr water, B.Cu at (87.6, 68.3)
- added G***: LOGO, logos:smartrv, B.Cu at (103.1, 67.1)
- added J1: 12v in, TerminalBlock_Phoenix:TerminalBlock_Phoenix_MKDS-1,5-2_1x02_P5.00mm_Horizontal, F.Cu at (121.5, 104.5)
- added J2: Programming Header, Connector_PinHeader_2.54mm:PinHeader_1x04_P2.54mm_Vertical, F.Cu at (83.4, 95.8)
- added J3: Valve Terminal, TerminalBlock_Phoenix:TerminalBlock_Phoenix_MKDS-1,5-3_1x03_P5.00mm_Horizontal, F.Cu at (121.5, 93.0)
- added J4: Temp Sensor, Connector_JST:JST_XH_S3B-XH-A-1_1x03_P2.50mm_Horizontal, F.Cu at (118.5, 67.5)
- added J5: Water Level Sensor, Connector_JST:JST_XH_S2B-XH-A-1_1x02_P2.50mm_Horizontal, F.Cu at (118.5, 76.5)
- added PS1: K7805-500R3, SamacSys_Parts:K7805500R3, F.Cu at (103.5, 99.5)
- added Q1: AO3400A, Package_TO_SOT_SMD:SOT-23, F.Cu at (92.8, 85.2)
- added R1: 47k, Resistor_SMD:R_0805_2012Metric, F.Cu at (89.9, 78.0)
- added R2: 470, Resistor_SMD:R_0805_2012Metric, F.Cu at (92.2, 78.0)
- added R3: 2k, Resistor_SMD:R_0805_2012Metric, F.Cu at (91.1, 90.7)
- added R4: 2k, Resistor_SMD:R_0805_2012Metric, F.Cu at (112.0, 105.9)
- added R5: 470, Resistor_SMD:R_0805_2012Metric, F.Cu at (84.1, 79.6)
- added R6: 4.7k, Resistor_SMD:R_0805_2012Metric, F.Cu at (84.1, 81.7)
- added R7: 10k, Resistor_SMD:R_0805_2012Metric, F.Cu at (84.1, 77.5)
- added R8: 10k, Resistor_SMD:R_0805_2012Metric, F.Cu at (84.1, 75.4)
- added Relay1: Relay, Relay_THT:Relay_SPDT_SANYOU_SRD_Series_Form_C, F.Cu at (96.5, 88.0)
- added S1: TS-1187A-B-A-B, SamacSys_Parts:TS1187ABAB, F.Cu at (100.5, 111.5)
- added S2: TS-1187A-B-A-B, SamacSys_Parts:TS1187ABAB, F.Cu at (112.0, 111.5)
- added U1: AMS1117-3.3, Package_TO_SOT_SMD:SOT-223-3_TabPin2, F.Cu at (90.4, 97.2)
- added U2: ESP32-WROOM-32D, RF_Module:ESP32-WROOM-32, F.Cu at (104.0, 68.5)
Routing:
- net GND: track 0.00 -> 120.2 mm, vias 0 -> 55
- net TX-ESP: track 0.00 -> 112.5 mm
- net RX-ESP: track 0.00 -> 107.7 mm, vias 0 -> 2
- net VDD33: track 0.00 -> 97.9 mm, vias 0 -> 1
- net Net-(R8-Pad2): track 0.00 -> 92.4 mm, vias 0 -> 6
- net Net-(R7-Pad2): track 0.00 -> 75.1 mm, vias 0 -> 4
- net +5V: track 0.00 -> 73.4 mm
- net ADC1: track 0.00 -> 61.2 mm
- net Temp: track 0.00 -> 58.2 mm, vias 0 -> 2
- net Net-(C5-Pad2): track 0.00 -> 55.1 mm, vias 0 -> 4
- net Net-(D5-Pad2): track 0.00 -> 40.3 mm
- net +12V: track 0.00 -> 37.6 mm
- net Net-(C1-Pad1): track 0.00 -> 14.7 mm
- net Valve: track 0.00 -> 11.4 mm
- net Net-(J3-Pad1): track 0.00 -> 11.3 mm
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- added copper zone on B.Cu, net GND
Other:
- board outline added: 49 x 67.5 mm
- board text added: "3v3"
- board text added: "3v3 GND TX RX"
- board text added: "9V-36V"
- board text added: "BOOT"
- board text added: "C"
- board text added: "D"
- board text added: "GND"
- board text added: "NC"
- board text added: "NO"
- board text added: "PWR"
- board text added: "RESET"
- board text added: "Tank Level"
- board text added: "Temp Sensor"
- board text added: "V IN"
- board text added: "Valve Control"
- board text added: "Water Tank Module V2"
- board text added: "robin@smartrv.uk"
