File: V2 SMD/Hardware/Water Tank Sensor V2.kicad_pcb (KiCad board)
At the start: 2 copper layers, 49 x 67.5 mm, 35 parts, among them J1 12v in, J2 Programming Header, J3 Valve Terminal, J4 Temp Sensor, J5 Water Level Sensor, Q1 AO3400A, U1 AMS1117-3.3, U2 ESP32-WROOM-32D

Commit message: Update
Routing:
- added copper zone on F.Cu, net GND
Changed lines of the file:
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@@
   (segment (start 94.742 114.808) (end 98.298 114.808) (width 0.2) (layer "B.Cu") (net 52))
   (segment (start 86.1 91.5) (end 86.1 93.6) (width 0.2) (layer "B.Cu") (net 52))
+  (zone (net 2) (net_name "GND") (layers F&B.Cu) (hatch edge 0.508)
+    (connect_pads (clearance 0.508))
+    (min_thickness 0.254) (filled_areas_thickness no)
+    (fill yes (thermal_gap 0.508) (thermal_bridge_width 0.508))
+    (polygon
+      (pts
+        (xy 128.5 59.1)
+        (xy 129 117.3)
+        (xy 79.4 117.3)
+        (xy 80.6 58.6)
+      )
+    )
+  )
   (zone (net 2) (net_name "GND") (layer "B.Cu") (hatch edge 0.508)
     (connect_pads (clearance 0.508))
